File: boards/tps63070-breakout/tps63070-breakout.kicad_sch (KiCad schematic)
At the start: 15 parts, among them J1 MODULE PINS, U1 TPS63070

Commit message: fix(tps63070-breakout): repair symbol-lib rename fallout and clear fab DRC
- ERC: point sym-lib-table at the renamed TPS63070-Buck-Boost.kicad_sym
  and update the embedded symbol + lib_id to TPS63070RNMR, matching the
  devkit (the PR's library rename had left this board referencing the
  deleted TPS630701 file)
- Mark embedded TPS63070 footprint as SMD (matches library fix)
- fab DRC: bump silkscreen reference text to 1.0mm/0.15mm (JLCPCB/PCBWay
  advanced minimums) and relocate C3's reference out of L1's silkscreen
- fab DRC: PCBWay advanced requires 0.15mm pad-to-silk clearance, which
  stock KiCad 0402 footprints violate; add repo-local Passives.pretty
  variants of R/C_0402_1005Metric without the body silk lines and switch
  the seven 0402 parts to them (schematic + board)

ERC, DRC, and both fab DRC targets (jlcpcb/pcbway 2-layer advanced) pass.

Co-Authored-By: Claude Fable 5 <noreply@anthropic.com>
Parts:
- C3, C4, C5: footprint Capacitor_SMD:C_0402_1005Metric -> Passives:C_0402_1005Metric
- R1, R2, R3, R4: footprint Resistor_SMD:R_0402_1005Metric -> Passives:R_0402_1005Metric
- U1: symbol TPS630701 Buck-Boost:TPS630701RNMR -> TPS63070 Buck-Boost:TPS63070RNMR
Changed lines of the file:
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@@
 			)
 		)
-		(property "Footprint" "Resistor_SMD:R_0402_1005Metric"
+		(property "Footprint" "Passives:R_0402_1005Metric"
 			(at 187.452 110.49 90)
 			(hide yes)
@@
 			)
 		)
-		(property "Footprint" "Capacitor_SMD:C_0402_1005Metric"
+		(property "Footprint" "Passives:C_0402_1005Metric"
 			(at 112.7252 93.98 0)
 			(hide yes)
@@
 			)
 		)
-		(property "Footprint" "Resistor_SMD:R_0402_1005Metric"
+		(property "Footprint" "Passives:R_0402_1005Metric"
 			(at 93.472 96.52 90)
 			(hide yes)
@@
 			)
 		)
-		(property "Footprint" "Resistor_SMD:R_0402_1005Metric"
+		(property "Footprint" "Passives:R_0402_1005Metric"
 			(at 200.152 107.95 90)
 			(hide yes)
@@
 			)
 		)
-		(property "Footprint" "Resistor_SMD:R_0402_1005Metric"
+		(property "Footprint" "Passives:R_0402_1005Metric"
 			(at 187.452 99.06 90)
 			(hide yes)
@@
 	)
 	(symbol
-		(lib_id "TPS630701 Buck-Boost:TPS630701RNMR")
+		(lib_id "TPS63070 Buck-Boost:TPS63070RNMR")
 		(at 144.78 109.22 0)
 		(unit 1)
@@
 			)
 		)
-		(property "Footprint" "Capacitor_SMD:C_0402_1005Metric"
+		(property "Footprint" "Passives:C_0402_1005Metric"
 			(at 176.2252 102.87 0)
 			(hide yes)
@@
 			)
 		)
-		(property "Footprint" "Capacitor_SMD:C_0402_1005Metric"
+		(property "Footprint" "Passives:C_0402_1005Metric"
 			(at 120.3452 127 0)
 			(hide yes)
