File: boards/esp32s3-devkit/esp32s3-devkit.kicad_pcb (KiCad board)
At the start: 4 copper layers, 59.3 x 38 mm, 37 parts, among them J1 Conn_01x17_Pin, J2 Conn_01x17_Pin, J3 USB_C_Receptacle_USB2.0_14P, Q1 Q_PMOS_GSD, SW1 ON/OFF, SW2 RESET, SW3 BOOT, U1 TPS630701RNMR, U2 ESP32-S3-WROOM-1, U3 USBLC6-2SC6

Commit message: fix(esp32s3-devkit): migrate J3 USB-C to 16P symbol and Connector_USB footprint.
Use KiCad Connector USB‑C USB2 16P (A8/B8 SH) with the KiCad Connector_USB HRO footprint, remove the duplicated HRO footprint lib, refresh PCB pad SH naming, and add a small migration helper script.
Parts:
- J3: footprint HRO_TypeC_USB:USB_C_Receptacle_HRO_TYPE-C-31-M-12 -> Connector_USB:USB_C_Receptacle_HRO_TYPE-C-31-M-12
Changed lines of the file:
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@@
 		)
 	)
-	(footprint "HRO_TypeC_USB:USB_C_Receptacle_HRO_TYPE-C-31-M-12"
+	(footprint "Connector_USB:USB_C_Receptacle_HRO_TYPE-C-31-M-12"
 		(layer "F.Cu")
 		(at 114.2875 114.2675 -90)
@@
 			(unit
 				(name "A")
-				(pins "S1" "A1" "A12" "B1" "B12" "A4" "A9" "B4" "B9" "A5" "B5" "A7" "B7"
-					"A6" "B6"
+				(pins "SH" "A1" "A4" "A5" "A6" "A7" "A8" "A9" "A12" "B1" "B4" "B5" "B6" "B7" "B8" "B9" "B12"
 				)
 			)
@@
 			(pintype "passive")
 		)
-		(pad "S1" thru_hole oval
+		(pad "SH" thru_hole oval
 			(at -4.32 -3.13 270)
 			(size 1 2.1)
@@
 			(remove_unused_layers no)
 		)
-		(pad "S1" thru_hole oval
+		(pad "SH" thru_hole oval
 			(at -4.32 1.05 270)
 			(size 1 1.6)
@@
 			(remove_unused_layers no)
 		)
-		(pad "S1" thru_hole oval
+		(pad "SH" thru_hole oval
 			(at 4.32 -3.13 270)
 			(size 1 2.1)
@@
 			(remove_unused_layers no)
 		)
-		(pad "S1" thru_hole oval
+		(pad "SH" thru_hole oval
 			(at 4.32 1.05 270)
 			(size 1 1.6)

Commit message: fix(esp32s3-devkit): pass standard DRC with USB net split and silk trim
Split merged VBUS/CC1 copper so CC1 is only J3 A5 and R10, route VBUS on
Net-(U3-VBUS), align J3 with the 16P schematic, and trim U2 silk inside the
board outline via a project RF_Module footprint override.
Parts:
- J3: value USB_C_Receptacle_USB2.0_14P -> USB_C_Receptacle_USB2.0_16P
Connections:
- C12 pad 1: Net-(J3-CC1) -> Net-(U3-VBUS)
- J3 pad A4: Net-(J3-CC1) -> Net-(U3-VBUS)
- J3 pad A8: (no net) -> unconnected-(J3-SBU1-PadA8)
- J3 pad A9: Net-(J3-CC1) -> Net-(U3-VBUS)
- J3 pad B4: Net-(J3-CC1) -> Net-(U3-VBUS)
- J3 pad B8: (no net) -> unconnected-(J3-SBU2-PadB8)
- J3 pad B9: Net-(J3-CC1) -> Net-(U3-VBUS)
- J3 pad SH: (no net) -> GND
- U3 pad 5: Net-(J3-CC1) -> Net-(U3-VBUS)
Routing:
- net Net-(U3-VBUS): track 0.00 -> 36.3 mm, vias 0 -> 3
- net Net-(J3-CC1): track 38.7 -> 2.38 mm, vias 3 -> 0
