File: boards/esp32s3-devkit/esp32s3-devkit.kicad_pcb (KiCad board)
At the start: 4 copper layers, 59.3 x 38 mm, 37 parts, among them J1 Conn_01x17_Pin, J2 Conn_01x17_Pin, J3 USB_C_Receptacle_USB2.0_16P, Q1 Q_PMOS_GSD, SW1 ON/OFF, SW2 RESET, SW3 BOOT, U1 TPS630701RNMR, U2 ESP32-S3-WROOM-1, U3 USBLC6-2SC6

Commit message: fix(esp32s3-devkit): use adjustable TPS63070 instead of fixed TPS630701 (#107)
* fix(esp32s3-devkit): use adjustable TPS63070 instead of fixed TPS630701

The schematic uses a resistor divider (R3=470k, R4=150k) on the FB pin
to regulate output to 3.3V, which requires the adjustable TPS63070RNMR.
The fixed TPS630701RNMR ignores the external divider and outputs 5V.

Renames the library symbol, schematic references, and PCB value to
TPS63070RNMR throughout. Also adds JLCPCB BOM and CPL assembly files.

* fix(esp32s3-devkit): replace SW1 with MK-12C03-G015 slide switch for JLCPCB availability

The original CK RS282G05A3 SPST switch (C2804704) is out of stock at
JLCPCB. Replace with G-Switch MK-12C03-G015 SPDT slide switch
(C2890358, ~4900 in stock) using KiCad's built-in
SW_SPDT_Shouhan_MSK12C02 footprint (same package family).

Schematic changes:
- SW1 symbol changed from SW_SPST to SW_SPDT
- Pin 2 (COM) connects to /PFET, pin 1 (Throw A) to /2-16v
- Pin 3 (Throw B) marked no-connect
- Footprint updated to Button_Switch_SMD:SW_SPDT_Shouhan_MSK12C02

BOM sync with user's JLCPCB part selections:
- D1/D3: C72043 -> C2286 (red LED, in stock)
- D2: C2928910 -> C493210 (BZT52B3V6S 3.6V Zener, in stock)
- SW1: C2804704 -> C2890358 (MK-12C03-G015 slide switch)

NOTE: PCB layout update required - user must run "Update PCB from
Schematic" in KiCad, place/route the new SW1 footprint, run DRC,
and regenerate Gerber files + CPL.

* fix(esp32s3-devkit): battery-only power-path and boot-reliability fixes

- Q1 (AO3401A): correct reverse-polarity orientation - schematic
  mirrored so drain faces battery, footprint rotated 180deg so pads
  land in the correct VBAT/PFET pours, gate rerouted via B.Cu hop,
  VBAT zone corner extended to enclose the drain pad
- Rename misleading '2-16v' net to 'VBAT_SW' (board is 3xAA powered)
- C11 EN delay cap 0.1uF -> 1uF (Espressif-recommended power-on delay)
- D2 3.6V zener marked DNP (leaks near knee at 3.3V, drains battery)
- Drop pcbway-4layer-adva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
Parts:
- C11: value 0.1µF -> 1µF
- SW1: value ON/OFF -> MK-12C03-G015; footprint Button_Switch_SMD:SW_SPST_CK_RS282G05A3 -> Button_Switch_SMD:SW_SPDT_Shouhan_MSK12C02
- U1: value TPS630701RNMR -> TPS63070RNMR
- moved D1 3.69 mm to (113.0, 92.7), turned to -90 degrees
- moved R1 3.69 mm to (113.0, 95.8)
- moved SW1 1.48 mm to (113.2, 103.3), turned to -90 degrees
- turned D3 to 180 degrees
- turned Q1 to -90 degrees
Connections:
- C1 pad 1: /2-16v -> /VBAT_SW
- C2 pad 1: /2-16v -> /VBAT_SW
- C3 pad 1: /2-16v -> /VBAT_SW
- D1 pad 1: Net-(D1-K) -> GND
- D1 pad 2: GND -> Net-(D1-A)
- D3 pad 1: Net-(D3-K) -> GND
- D3 pad 2: GND -> Net-(D3-A)
- Q1 pad 2: /VBAT -> /PFET
- Q1 pad 3: /PFET -> /VBAT
- R1 pad 1: /2-16v -> /VBAT_SW
- R1 pad 2: Net-(D1-K) -> Net-(D1-A)
- R2 pad 1: /2-16v -> /VBAT_SW
- R6 pad 2: Net-(D3-K) -> Net-(D3-A)
- SW1 pad 1: /PFET -> /VBAT_SW
- SW1 pad 2: /2-16v -> /PFET
- U1 pad 12: /2-16v -> /VBAT_SW
- U1 pad 13: /2-16v -> /VBAT_SW
Routing:
- net /2-16v: track 5.33 -> 0.00 mm
- net Net-(Q1-G): track 2.02 -> 7.01 mm, vias 0 -> 2
- net GND: track 71.1 -> 75.7 mm, vias 53 -> 57
- net Net-(D1-K): track 1.80 -> 0.00 mm
- net Net-(D1-A): track 0.00 -> 1.80 mm
- net Net-(D3-K): track 1.55 -> 0.00 mm
- net Net-(D3-A): track 0.00 -> 1.55 mm
- added copper zone on F.Cu, net /VBAT_SW
- removed copper zone on F.Cu, net /2-16v

Commit message: test(esp32s3-devkit): add design validation, battery-range SPICE, and bring-up plan
Board-level test coverage for the battery-powered devkit ahead of fab:

- checks.yml: design-intent validation (make validate) — pins all 31
  components incl. Q1=AO3401A and U2=ESP32-S3-WROOM-1-N16 (values aligned
  with the JLCPCB BOM), required nets, input/output capacitance budgets,
  BOM hygiene, and the TPS63070 FB divider math (0.8V ref, 3.3V ±2% —
  guards the exact fixed-vs-adjustable bug PR #107 fixed)
- sim.yml + sim/: opt-in SPICE (make sim-board / CI spice-board) sweeping
  the 3xAA range 4.8V -> 3.6V (buck-boost transition) -> 3.0V (end-of-life)
  with 0.5A WiFi-TX load bursts, plus a cold-start-at-3.0V secondary pass;
  13 bounded measures with committed baseline. The TI model is quasi-ideal
  (documented in sim.yml), so these act as topology regressions — a
  miswired divider or dead rail fails loudly
- schematic: add Sim.* subckt mapping to U1 instance; exclude non-electrical
  parts (module, USB, switches, LEDs, PMOS, connectors) from simulation;
  footprint_symbol_field_mismatch set to ignore to match the breakout's
  convention for symbol-only Sim fields
- docs/bringup.md: bench-test checklist for first articles — smoke checks,
  reverse-battery, brown-out sweep, USB flashing on battery (incl. weak-pack
  boot strapping), WiFi soak on tired cells, deep-sleep current record
- tests: sim discovery now expects esp32s3-devkit to be opted in

make validate, make check, and the full SPICE suite pass locally.

Co-Authored-By: Claude Fable 5 <noreply@anthropic.com>
Parts:
- Q1: value Q_PMOS_GSD -> AO3401A
- U2: value ESP32-S3-WROOM-1 -> ESP32-S3-WROOM-1-N16
Changed lines of the file:
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@@
 			)
 		)
-		(property "Value" "ESP32-S3-WROOM-1"
+		(property "Value" "ESP32-S3-WROOM-1-N16"
 			(at 0 14.6 270)
 			(unlocked yes)
@@
 			)
 		)
-		(property "Value" "Q_PMOS_GSD"
+		(property "Value" "AO3401A"
 			(at 0 2.4 270)
 			(layer "F.Fab")
