File: boards/esp32s3-devkit/esp32s3-devkit.kicad_sch (KiCad schematic)
At the start: 37 parts, among them J1 Conn_01x17_Pin, J2 Conn_01x17_Pin, J3 USB_C_Receptacle_USB2.0_16P, Q1 Q_PMOS_GSD, SW1 MK-12C03-G015, SW2 RESET, SW3 BOOT, U1 TPS63070RNMR, U2 ESP32-S3-WROOM-1, U3 USBLC6-2SC6

Commit message: fix(esp32s3-devkit): battery-only power-path and boot-reliability fixes
- Q1 (AO3401A): correct reverse-polarity orientation - schematic
  mirrored so drain faces battery, footprint rotated 180deg so pads
  land in the correct VBAT/PFET pours, gate rerouted via B.Cu hop,
  VBAT zone corner extended to enclose the drain pad
- Rename misleading '2-16v' net to 'VBAT_SW' (board is 3xAA powered)
- C11 EN delay cap 0.1uF -> 1uF (Espressif-recommended power-on delay)
- D2 3.6V zener marked DNP (leaks near knee at 3.3V, drains battery)
- Drop pcbway-4layer-advanced fab target (module thermal vias can
  never pass its min pad hole rule; JLCPCB is the shipping target)
- README: battery-only power (USB is data-only by design), corrected
  refdes table, C3 6.3V input-voltage note, first-flash procedure

Note: zone fills need refill in KiCad; fab outputs regenerate in CI.
Parts:
- C11: value 0.1µF -> 1µF
- D2: now not fitted; now left out of the parts list
Connections:
- net PFET: no longer Q1.3 (D)
- net VBAT: no longer Q1.2 (S)
- net at R11.1: no longer Q1.1 (G)
- net 2-16v renamed VBAT_SW
Changed lines of the file:
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@@
 	)
 	(no_connect
-		(at 106.68 134.62)
+		(at 67.31 49.53)
 	)
 	(no_connect
-		(at 167.64 146.05)
+		(at 106.68 134.62)
 	)
 	(no_connect
-		(at 67.31 49.53)
+		(at 167.64 146.05)
 	)
 	(wire
@@
 	(wire
 		(pts
-			(xy 67.31 44.45) (xy 67.31 46.99)
-		)
-		(stroke
-			(width 0)
-			(type default)
-		)
-	)
-	(wire
-		(pts
 			(xy 67.31 46.99) (xy 72.39 46.99)
 		)
@@
 	(wire
 		(pts
+			(xy 67.31 44.45) (xy 67.31 46.99)
+		)
+		(stroke
+			(width 0)
+			(type default)
+		)
+	)
+	(wire
+		(pts
 			(xy 184.15 110.49) (xy 190.5 110.49)
 		)
@@
 		)
 	)
-	(label "2-16v"
+	(label "VBAT_SW"
 		(at 68.58 46.99 0)
 		(effects
@@
 		(body_style 1)
 		(exclude_from_sim no)
-		(in_bom yes)
+		(in_bom no)
 		(on_board yes)
 		(in_pos_files yes)
-		(dnp no)
+		(dnp yes)
 		(fields_autoplaced yes)
 		(property "Reference" "D2"
@@
 		(lib_id "Transistor_FET:Q_PMOS_GSD")
 		(at 46.99 44.45 270)
+		(mirror x)
 		(unit 1)
 		(body_style 1)
@@
 			)
 		)
-		(property "Value" "0.1µF"
+		(property "Value" "1µF"
 			(at 65.024 109.474 0)
 			(show_name no)
