File: boards/esp32s3-devkit-5v/esp32s3-devkit-5v.kicad_sch (KiCad schematic)
At the start: 78 parts, among them J1 Conn_01x02_Pin, J2 USB_C_Receptacle_USB2.0_16P, J3 Conn_01x02_Pin, J4 Conn_01x04_Pin, Q1 AO3401A, Q2 AO3401A, Q3 MMBT3904, SW1 MK-12C03-G015, SW2 RESET, SW3 BOOT, SW4 SW_Push, SW5 SW_Push, SW6 SW_Push, SW7 SW_Push, U1 TPS63070RNMR, U2 TPS63070RNMR, U3 ESP32-S3-WROOM-1-N16, U4 USBLC6-2SC6, U5 RV-3028-C7, U6 MAX98357A

Commit message: feat(esp32s3-devkit-5v): amp-local 5V caps + ERC cleanup to one benign note
Erik added the amp-local cap cluster at U6 (drawn there so layout places it
at the amp, not the converter): C26 100uF burst reservoir, C27 10uF mid,
C28 0.1uF HF decoupling — 5V rail now 186uF total, sized against the
volume-induced brownouts this board exists to fix. Also cleared the 16 stray
wire stubs; ERC is down to the single benign U6 thermal-pad note.

checks.yml: add C26-C28 (5V budget min raised to 150uF, C28 in decoupling),
and correct the C21 comment — it's the RTC-block 3v3 bulk, not a misplaced
amp cap (earlier note was wrong).

Still queued (needs KiCad closed): footprints for C26-C28 and
exclude_from_sim on the 12 model-less rev-2 parts (the SPICE-crash fix).

Co-Authored-By: Claude Opus 4.8 <noreply@anthropic.com>
Parts:
- added C26: 100µF, Capacitor_SMD:C_0402_1005Metric, symbol Device:C
- added C27: 10µF, Capacitor_SMD:C_0402_1005Metric, symbol Device:C
- added C28: 0.1µF, Capacitor_SMD:C_0402_1005Metric, symbol Device:C
Connections:
- net 5v: now also C26.1, C27.1, C28.1
- net GND: now also C26.2, C27.2, C28.2

Commit message: fix(esp32s3-devkit-5v): sim-exclude model-less parts; correct amp-cap footprints
- exclude_from_sim on the 12 rev-2 parts with no SPICE model (RTC, amp, OLED
  switch PMOS+NPN, RGB LED, 4 buttons, 3 connectors). The schematic's SPICE
  export now contains only the power path (R/L/C + both TPS63070 subckts),
  which is what crashed ngspice in CI — every measure read "(missing)".
- C26 100uF 0402 doesn't exist -> 1206; C27 10uF 0402 is the 6.3V-rated
  C15525 trap the board README forbids on the 5V rail -> 0805. C28 0402 kept.

Validator PASS. ERC at the single excluded-pending U6 pad note.

Co-Authored-By: Claude Opus 4.8 <noreply@anthropic.com>
Parts:
- C26: footprint Capacitor_SMD:C_0402_1005Metric -> Capacitor_SMD:C_1206_3216Metric
- C27: footprint Capacitor_SMD:C_0402_1005Metric -> Capacitor_SMD:C_0805_2012Metric
