File: boards/esp32s3-devkit-5v/esp32s3-devkit-5v.kicad_sch (KiCad schematic)
At the start: 53 parts, among them J1 Conn_01x17_Pin, J2 Conn_01x17_Pin, J3 USB_C_Receptacle_USB2.0_16P, Q1 AO3401A, SW1 MK-12C03-G015, SW2 RESET, SW3 BOOT, U1 TPS63070RNMR, U2 ESP32-S3-WROOM-1-N16, U2 TPS63070RNMR, U3 USBLC6-2SC6

Commit message: wip(esp32s3-devkit-5v): add RV-3028-C7 RTC subcircuit + resolve annotation/flag cleanup
Adds the real-time clock (U5, RV-3028-C7, Package_SON C7 SON-8) for the rev-2
deep-sleep alarm wake. Verified against cube_browns.ino pin map:

  /INT -> GPIO1   (open-drain, 10k pull-up R18) — deep-sleep wake
  SCL  -> GPIO9   (4.7k pull-up R16)
  SDA  -> GPIO8   (4.7k pull-up R17)
  VDD, VBACKUP -> 3V3   (VBACKUP tied to VDD — no separate backup; Cube re-syncs
                         time from the Beacon over ESP-NOW, so a battery swap
                         losing the count is fine. Leave trickle charger OFF.)
  VSS, EVI -> GND ;  CLKOUT -> NC ;  100nF decoupling on VDD

I2C pull-ups: exactly one pair on the shared bus (SDA/SCL) — do NOT add a second
pair when the OLED lands. RTC addr 0x52, no conflict with the OLED's 0x3C.

Also folded in the earlier schematic cleanup: annotation resolved (no dupes),
PWR_FLAGs down to the clean set (VBAT / VBAT_SW / GND), stray wire removed.

JLC part for the BOM: LCSC C3019759 (RV-3028-C7 TA-QC) — in stock, SMT-assemblable
on Economic+Standard, Extended part (one-time feeder fee). Package SMD3215-8P
matches the assigned footprint.

Still WIP / ERC not clean: J2 battery connector pins float (connector being
reworked), and the amp + display + display-PMOS blocks are still to come.

Co-Authored-By: Claude Opus 4.8 <noreply@anthropic.com>
Parts:
- removed D1, D?: LED, LED_SMD:LED_0603_1608Metric, symbol Device:LED
- removed D2: 3.6v, Diode_SMD:D_SOD-323, symbol Device:D_Zener
- removed R1, R?: 1kΩ, Resistor_SMD:R_0402_1005Metric, symbol Device:R
- added C21: 100µF, symbol Device:C
- added J1: Conn_01x02_Pin, Connector_JST:JST_PH_B2B-PH-SM4-TB_1x02-1MP_P2.00mm_Vertical, symbol Connector:Conn_01x02_Pin
- added R16, R17: 4.7kΩ, symbol Device:R
- added R18: 10kΩ, symbol Device:R
- added U5: RV-3028-C7, Package_SON:MicroCrystal_C7_SON-8_1.5x3.2mm_P0.9mm, symbol Timer_RTC:RV-3028-C7
- gave numbers to parts that had none: 13
- renumbered C9 to C17, C10 to C18, C11 to C19, C12 to C20, J1 to J2, J2 to J3, J3 to J4, R11 to R1, R6 to R11, R7 to R12, R8 to R13, R9 to R14, R10 to R15, R2 to R3, R3 to R4, R4 to R5, R5 to R6, U2 to U3, U3 to U4
Connections:
- net 3v3: now also C21.1, R16.2, R17.2, R18.2, U5.6 (VBACKUP), U5.7 (VDD)
- net GND: now also C21.2, J1.2 (Pin_2), U5.5 (VSS), U5.8 (EVI); no longer J2.1 (Pin_1)
- net GPIO1: now also R18.1, U5.2 (~{INT})
- net GPIO8: now also R17.1, U5.4 (SDA)
- net GPIO9: now also R16.1, U5.3 (SCL)
- net VBAT: now also J1.1 (Pin_1); no longer J2.2 (Pin_2)
- net at C20.1, J4.A4 (VBUS), J4.A9 (VBUS)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: no longer J4.A5 (CC1), R15.1
- new net: J4.A5 (CC1), R15.1
- no-connect marks 6 -> 7
Other:
- note added: "TODO: - Add RTC - Add Amp - Add Display + PMOSFET"
- note removed: "TODO: - Add battery connector - Update ? Values - Add RTC - Add Amp - Add Display + PMOSFET"
- moved on the sheet: C1, C10, C11, C12, C13, C14, C15, C16, C17, C18, C19, C2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

Commit message: feat(esp32s3-devkit-5v): GPIO-gate the 5V boost enable (BOOST_EN on GPIO18)
The 5V stage (U2) was always-on with EN strapped to VBAT_SW. Put it under
firmware control so the amp rail can be shed during battery sag — matches
cube_browns.ino `BOOST_EN 18`.

- U2 EN (pin 14) -> GPIO18, with R19 100k pulldown to GND so the rail defaults
  OFF at boot/reset/deep-sleep until firmware drives GPIO18 high.
- U2 PS/SYNC (pin 1) correctly un-strapped from EN (they shared a pull-up on the
  U1-copied block) and kept pulled to VBAT_SW via R7 -> forced-PWM on the 5V rail.
  Fine here: the rail is gated off when idle, and PWM gives better transient
  response for the amp's ESP-NOW-burst loads.

U1 (3.3V) left as-is per design discussion. ERC unchanged: only the deferred J2
battery-connector pins remain.

Co-Authored-By: Claude Opus 4.8 <noreply@anthropic.com>
Parts:
- added R19: 100kΩ, symbol Device:R
Connections:
- net GND: now also R19.2
- net GPIO18: now also U2.14 (EN), R19.1
- net at R7.2, U2.1 (PS_SYNC): no longer U2.14 (EN)
- net at J4.A5 (CC1), R15.1: now also C20.1, J4.A4 (VBUS), J4.A9 (VBUS), J4.B4 (VBUS), J4.B9 (VBUS), U4.5 (VBUS)
Other:
- moved on the sheet: C20, C21, J2, J3, J4, R14, R15, R16, R17, R18, U4, U5

Commit message: feat(esp32s3-devkit-5v): rev-2 schematic — amp, display, RTC control, front panel (#121)
* wip(esp32s3-devkit-5v): add audio amp + power-gated display blocks

Two new functional blocks, both traced and verified against cube_browns.ino:

Audio amp (U6, MAX98357A, JLC C910544):
- I2S: DIN->GPIO17, BCLK->GPIO15, LRCLK->GPIO16
- SD_MODE->GPIO21 + 100k pulldown (default-off), GAIN->GND (12 dB)
- VDD on the 5V rail, OUTP/OUTN -> speaker (JST-PH), NC pins flagged

Display power-gate (matches the breadboard PMOS + 2N3904):
- High-side PMOS load switch (Q2 AO3401A) on the 3V3 rail, gated by an
  MMBT3904 (Q3) inverter so GPIO7 HIGH = display ON (matches PIN_OLED_PWR)
- R21 100k gate pull-up, R22 10k base (from GPIO7), R23 100k base pull-down
- 4-pin OLED connector (J4): switched VDD / GND / SCL->GPIO9 / SDA->GPIO8,
  reusing the shared I2C bus (no new pull-ups; addr 0x3C, no RTC conflict)

Also resolved the R19 duplicate refdes (amp + boost pulldowns now unique).

Still WIP: buttons + RGB LED to come; 18 unused GPIOs need no-connect flags,
plus a few stray wire stubs and the benign U6 thermal-pad ERC note.

Co-Authored-By: Claude Opus 4.8 <noreply@anthropic.com>

* feat(esp32s3-devkit-5v): add 4 front-panel buttons

Mode/Vol+/Vol-/4th on GPIO4/5/6/10 (matches cube_browns.ino PIN_MODE/VOL_UP/
VOL_DOWN; GPIO10 is RTC-capable so the 4th can also wake from deep sleep).

Each button: SW_Push (TS-1187A) to the GPIO node + GND, 10k pull-up to 3v3
(robust idle level for EXT1 deep-sleep wake), 100nF debounce to GND. Active-low,
matching the firmware's INPUT_PULLUP.

Added programmatically via kicad-skip, grid-aligned; connectivity by local labels
(this sheet wires everything, incl. GND/3v3, with local labels). ERC adds no new
violations. Positions are functional — hand-tidy the layout as desired.

Co-Authored-By: Claude Opus 4.8 <noreply@anthropic.com>

* feat(esp32s3-devkit-5v): add RGB status LED (D4, common cathode)

Device:LED_RGBK on GPIO38/39/40 (PWM via LEDC), cathode to GND:
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
Parts:
- removed J2, J3: Conn_01x17_Pin, Connector_PinHeader_2.54mm:PinHeader_1x17_P2.54mm_Vertical, symbol Connector:Conn_01x17_Pin
- added C22, C23, C24, C25, C28: 0.1µF, Capacitor_SMD:C_0402_1005Metric, symbol Device:C
- added C26: 100µF, Capacitor_SMD:C_1206_3216Metric, symbol Device:C
- added C27: 10µF, Capacitor_SMD:C_0805_2012Metric, symbol Device:C
- added D4: LED_RGBK, LED_SMD:LED_RGB_Wuerth-PLCC4_3.2x2.8mm_150141M173100, symbol Device:LED_RGBK
- added J3: Conn_01x02_Pin, Connector_JST:JST_PH_B2B-PH-SM4-TB_1x02-1MP_P2.00mm_Vertical, symbol Connector:Conn_01x02_Pin
- added J4: Conn_01x04_Pin, Connector_PinHeader_2.54mm:PinHeader_1x04_P2.54mm_Vertical, symbol Connector:Conn_01x04_Pin
- added Q2: AO3401A, Package_TO_SOT_SMD:SOT-23, symbol Transistor_FET:AO3401A
- added Q3: MMBT3904, Package_TO_SOT_SMD:SOT-23, symbol Transistor_BJT:MMBT3904
- added R20, R21, R23: 100kΩ, Resistor_SMD:R_0402_1005Metric, symbol Device:R
- added R22, R24, R25, R26, R27: 10kΩ, Resistor_SMD:R_0402_1005Metric, symbol Device:R
- added R28: 330Ω, Resistor_SMD:R_0402_1005Metric, symbol Device:R
- added R29, R30: 150Ω, Resistor_SMD:R_0402_1005Metric, symbol Device:R
- added SW4, SW5, SW6, SW7: SW_Push, Button_Switch_SMD:SW_Push_1P1T_XKB_TS-1187A, symbol Switch:SW_Push
- added U6: MAX98357A, Package_DFN_QFN:TQFN-16-1EP_3x3mm_P0.5mm_EP1.23x1.23mm, symbol Audio:MAX98357A
- C21: footprint (none) -> Capacitor_SMD:C_1206_3216Metric
- R16, R17, R18, R19: footprint (none) -> Resistor_SMD:R_0402_1005Metric
- renumbered J4 to J2
Connections:
- net 3v3: now also Q2.2 (S), R21.1, R24.1, R25.1, R26.1, R27.1
- net 5v: now also C26.1, C27.1, C28.1, U6.7 (VDD), U6.8 (VDD)
- net GND: now also C22.2, C23.2, C24.2, C25.2, C26.2, C27.2, C28.2, D4.4 (K), J4.1 (Pin_1), Q3.2 (E), R20.2, R23.2, SW4.1, SW5.1, SW6.1, SW7.1, U6.11 (GND), U6.15 (GND), U6.17 (PAD), U6.2 (GAIN_SLOT), U6.3 (GND)
- net GPIO10: now also C25.1, R27.2, SW7.2
- net GPIO15: now also U6.16 (BCLK)
- net GPIO16: now also U6.14 (LRCLK)
- net GPIO17: now also U6.1 (DIN)
- net GPIO21: now also R20.1, U6.4 (~{SD_MODE})
- net GPIO38: now also R28.2
- net GPIO39: now also R29.2
- net GPIO4: now also C22.1, R24.2, SW4.2
- net GPIO40: now also R30.2
- net GPIO5: now also C23.1, R25.2, SW5.2
- net GPIO6: now also C24.1, R26.2, SW6.2
- net GPIO7: now also R22.2
- net GPIO8: now also J4.4 (Pin_4)
- net GPIO9: now also J4.3 (Pin_3)
- net GPIO11: no longer names the net of U3.19 (IO11)
- net GPIO12: no longer names the net of U3.20 (IO12)
- net GPIO13: no longer names the net of U3.21 (IO13)
- net GPIO14: no longer names the net of U3.22 (IO14)
- net GPIO2: no longer names the net of U3.38 (IO2)
- net GPIO3: no longer names the net of U3.15 (IO3)
- net GPIO41: no longer names the net of U3.34 (IO41)
- net GPIO42: no longer names the net of U3.35 (IO42)
- net GPIO45: no longer names the net of U3.26 (IO45)
- net GPIO46: no longer names the net of U3.16 (IO46)
- net GPIO47: no longer names the net of U3.24 (IO47)
- net GPIO48: no longer names the net of U3.25 (IO48)
- net RX: no longer names the net of U3.36 (RXD0)
- net TX: no longer names the net of U3.37 (TXD0)
- new net: Q2.1 (G), Q3.3 (C), R21.2
- new net: D4.3 (BA), R30.1
- new net: Q3.1 (B), R22.1, R23.1
- new net: D4.2 (GA), R29.1
- new net: D4.1 (RA), R28.1
- new net VCC: J4.2 (Pin_2), Q2.3 (D)
- new net speaker +: J3.2 (Pin_2), U6.9 (OUTP)
- new net speaker -: J3.1 (Pin_1), U6.10 (OUTN)
- no-connect marks 7 -> 21
Other:
- note removed: "TODO: - Add RTC - Add Amp - Add Display + PMOSFET"
- moved on the sheet: C1, C10, C11, C12, C13, C14, C15, C16, C17, C18, C19, C2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
